File: schem/v2/v2.kicad_sch (KiCad schematic)
At the start: 3 parts, among them U1 DOIT-ESP32-DEVKIT-V1

Commit message: v2 schem+pcb connected
Parts:
- RV1: value R_Potentiometer -> 10k; footprint (none) -> Potentiometer_THT:Potentiometer_Bourns_3296W_Vertical
Connections:
- net at RV1.1: now also DS1.15 (LED(+)), DS1.2 (VDD), U1.18 (VIN)
- net at RV1.2: now also DS1.3 (VO)
- net GND: now reaches RV1.3
- net GND: now also DS1.1 (VSS), DS1.16 (LED(-)), DS1.5 (R/W), U1.17 (GND)
- net at DS1.11 (D4): now also U1.32 (GPIO21_I2C-SDA)
- net at DS1.12 (D5): now also U1.31 (GPIO19_VSPI-MISO)
- net at DS1.13 (D6): now also U1.30 (GPIO18_VSPI-CLK)
- net at DS1.14 (D7): now also U1.29 (GPIO5_VSPI-CS0)
- net at DS1.4 (RS): now also U1.36 (GPIO23_VSPI-MOSI)
- net at DS1.6 (E): now also U1.35 (GPIO22_I2C-SCL)
